Commit message: Added robot description

File: src/tank_description/urdf/robot.urdf.xacro (robot description, xacro)
@@ -1,5 +1,5 @@
 <?xml version="1.0"?>
-<robot name="xiaor_geek_tank">
-  <!-- Main chassis -->
+<robot name="xiaor_geek_tank_colored">
+  <!-- Main chassis (raised) -->
   <link name="base_link">
     <visual>
@@ -7,5 +7,6 @@
         <box size="0.30 0.20 0.05"/> <!-- 30cm x 20cm x 5cm -->
       </geometry>
-      <material name="green">
+      <origin xyz="0 0 0.05"/> <!-- raise it above the tracks -->
+      <material name="silver">
         <color rgba="0.7 0.7 0.7 1.0"/>
       </material>
@@ -15,8 +16,9 @@
         <box size="0.30 0.20 0.05"/>
       </geometry>
+      <origin xyz="0 0 0.05"/>
     </collision>
     <inertial>
       <mass value="2.0"/>
-      <origin xyz="0 0 0"/>
+      <origin xyz="0 0 0.05"/>
       <inertia ixx="0.1" ixy="0.0" ixz="0.0"
                iyy="0.1" iyz="0.0"
@@ -30,5 +32,5 @@
         <box size="0.30 0.03 0.05"/>
       </geometry>
-      <material name="blue">
+      <material name="black">
         <color rgba="0.1 0.1 0.1 1.0"/>
       </material>
@@ -46,5 +48,7 @@
         <box size="0.30 0.03 0.05"/>
       </geometry>
-      <material name="red"/>
+      <material name="black_track">
+        <color rgba="0.15 0.15 0.15 1.0"/>
+      </material>
     </visual>
   </link>
@@ -60,6 +64,6 @@
         <cylinder radius="0.03" length="0.02"/>
       </geometry>
-      <material name="dark_gray">
-        <color rgba="0.2 0.2 0.2 1.0"/>
+      <material name="red_wheel">
+        <color rgba="1.0 0.2 0.2 1.0"/>
       </material>
     </visual>
@@ -68,5 +72,5 @@
     <parent link="base_link"/>
     <child link="left_wheel"/>
-    <origin xyz="-0.11 0.115 -0.025" rpy="0 1.5708 0"/>
+    <origin xyz="-0.11 0.13 0" rpy="1.5708 0 0"/>
   </joint>
   <!-- Right drive wheel -->
@@ -76,5 +80,7 @@
         <cylinder radius="0.03" length="0.02"/>
       </geometry>
-      <material name="dark_gray"/>
+      <material name="red_wheel">
+        <color rgba="1.0 0.2 0.2 1.0"/>
+      </material>
     </visual>
   </link>
@@ -82,5 +88,5 @@
     <parent link="base_link"/>
     <child link="right_wheel"/>
-    <origin xyz="-0.11 -0.115 -0.025" rpy="0 1.5708 0"/>
+    <origin xyz="-0.11 -0.13 0" rpy="1.5708 0 0"/>
   </joint>
   <!-- Left idler wheel -->
@@ -90,6 +96,6 @@
         <cylinder radius="0.03" length="0.02"/>
       </geometry>
-      <material name="gray">
-        <color rgba="0.3 0.3 0.3 1.0"/>
+      <material name="green_idler">
+        <color rgba="0.2 1.0 0.2 1.0"/>
       </material>
     </visual>
@@ -98,5 +104,5 @@
     <parent link="base_link"/>
     <child link="left_idler"/>
-    <origin xyz="0.11 0.115 -0.025" rpy="0 1.5708 0"/>
+    <origin xyz="0.11 0.13 0" rpy="1.5708 0 0"/>
   </joint>
   <!-- Right idler wheel -->
@@ -106,5 +112,7 @@
         <cylinder radius="0.03" length="0.02"/>
       </geometry>
-      <material name="gray"/>
+      <material name="green_idler">
+        <color rgba="0.2 1.0 0.2 1.0"/>
+      </material>
     </visual>
   </link>
@@ -112,5 +120,5 @@
     <parent link="base_link"/>
     <child link="right_idler"/>
-    <origin xyz="0.11 -0.115 -0.025" rpy="0 1.5708 0"/>
+    <origin xyz="0.11 -0.13 0" rpy="1.5708 0 0"/>
   </joint>
 </robot>

Commit message: added robot description

File: src/tank_description/urdf/robot.urdf.xacro (robot description, xacro)
@@ -5,7 +5,27 @@
     <visual>
       <geometry>
-        <box size="0.30 0.20 0.05"/> <!-- 30cm x 20cm x 5cm -->
+        <box size="0.30 0.14 0.05"/> <!-- 30cm x 14cm x 5cm -->
       </geometry>
       <origin xyz="0 0 0.05"/> <!-- raise it above the tracks -->
+      <material name="silver">
+        <color rgba="0.7 0.7 0.7 1.0"/>
+      </material>
+    </visual>
+    <!-- Middle square -->
+    <visual>
+      <geometry>
+        <box size="0.16 0.14 0.05"/>
+      </geometry>
+      <origin xyz="0.07 0 0.10"/> <!-- sits on top of bottom rectangle -->
+      <material name="BlueTop">
+        <color rgba="0.2 0.2 0.8 1"/>
+      </material>
+    </visual>
+    <!-- Top square -->
+    <visual>
+      <geometry>
+        <box size="0.16 0.14 0.05"/>
+      </geometry>
+      <origin xyz="0.07 0 0.15"/> <!-- sits on top of bottom rectangle -->
       <material name="silver">
         <color rgba="0.7 0.7 0.7 1.0"/>
@@ -61,32 +81,28 @@
   <link name="left_wheel">
     <visual>
-      <geometry>
-        <cylinder radius="0.03" length="0.02"/>
-      </geometry>
-      <material name="red_wheel">
-        <color rgba="1.0 0.2 0.2 1.0"/>
-      </material>
+      <geometry><cylinder radius="0.03" length="0.02"/></geometry>
+      <origin rpy="1.5708 0 0"/>   <!-- makes the cylinder look like a wheel -->
+      <material name="red_wheel"><color rgba="1.0 0.2 0.2 1.0"/></material>
     </visual>
   </link>
-  <joint name="left_wheel_joint" type="fixed">
+  <joint name="left_wheel_joint" type="continuous">
     <parent link="base_link"/>
     <child link="left_wheel"/>
-    <origin xyz="-0.11 0.13 0" rpy="1.5708 0 0"/>
+    <origin xyz="-0.11 0.13 0"/>
+    <axis xyz="0 1 0"/>
   </joint>
   <!-- Right drive wheel -->
   <link name="right_wheel">
     <visual>
-      <geometry>
-        <cylinder radius="0.03" length="0.02"/>
-      </geometry>
-      <material name="red_wheel">
-        <color rgba="1.0 0.2 0.2 1.0"/>
-      </material>
+      <geometry><cylinder radius="0.03" length="0.02"/></geometry>
+      <origin rpy="1.5708 0 0"/>
+      <material name="red_wheel"><color rgba="1.0 0.2 0.2 1.0"/></material>
     </visual>
   </link>
-  <joint name="right_wheel_joint" type="fixed">
+  <joint name="right_wheel_joint" type="continuous">
     <parent link="base_link"/>
     <child link="right_wheel"/>
-    <origin xyz="-0.11 -0.13 0" rpy="1.5708 0 0"/>
+    <origin xyz="-0.11 -0.13 0"/>
+    <axis xyz="0 1 0"/>
   </joint>
   <!-- Left idler wheel -->

Commit message: updated xacro to swap the stack to the back of the robot

File: src/tank_description/urdf/robot.urdf.xacro (robot description, xacro)
@@ -12,20 +12,20 @@
       </material>
     </visual>
-    <!-- Middle square -->
+    <!-- Middle block (moved to -X so it looks like the rear) -->
     <visual>
       <geometry>
         <box size="0.16 0.14 0.05"/>
       </geometry>
-      <origin xyz="0.07 0 0.10"/> <!-- sits on top of bottom rectangle -->
+      <origin xyz="-0.07 0 0.10"/> <!-- was +0.07; negative puts it behind the base center -->
       <material name="BlueTop">
         <color rgba="0.2 0.2 0.8 1"/>
       </material>
     </visual>
-    <!-- Top square -->
+    <!-- Top block (also moved to -X) -->
     <visual>
       <geometry>
         <box size="0.16 0.14 0.05"/>
       </geometry>
-      <origin xyz="0.07 0 0.15"/> <!-- sits on top of bottom rectangle -->
+      <origin xyz="-0.07 0 0.15"/>
       <material name="silver">
         <color rgba="0.7 0.7 0.7 1.0"/>
@@ -38,4 +38,5 @@
       <origin xyz="0 0 0.05"/>
     </collision>
+    <!-- Simple inertial; tune as needed -->
     <inertial>
       <mass value="2.0"/>
@@ -46,5 +47,5 @@
     </inertial>
   </link>
-  <!-- Left track -->
+  <!-- Left track (fixed visual) -->
   <link name="left_track">
     <visual>
@@ -62,5 +63,5 @@
     <origin xyz="0 0.115 0"/>
   </joint>
-  <!-- Right track -->
+  <!-- Right track (fixed visual) -->
   <link name="right_track">
     <visual>
@@ -78,9 +79,9 @@
     <origin xyz="0 -0.115 0"/>
   </joint>
-  <!-- Left drive wheel -->
+  <!-- Left drive wheel (continuous around +Y) -->
   <link name="left_wheel">
     <visual>
       <geometry><cylinder radius="0.03" length="0.02"/></geometry>
-      <origin rpy="1.5708 0 0"/>   <!-- makes the cylinder look like a wheel -->
+      <origin rpy="1.5708 0 0"/>   <!-- makes cylinder look like a wheel -->
       <material name="red_wheel"><color rgba="1.0 0.2 0.2 1.0"/></material>
     </visual>
@@ -92,5 +93,5 @@
     <axis xyz="0 1 0"/>
   </joint>
-  <!-- Right drive wheel -->
+  <!-- Right drive wheel (continuous around +Y) -->
   <link name="right_wheel">
     <visual>
@@ -106,13 +107,10 @@
     <axis xyz="0 1 0"/>
   </joint>
-  <!-- Left idler wheel -->
+  <!-- Left idler (fixed) -->
   <link name="left_idler">
     <visual>
-      <geometry>
-        <cylinder radius="0.03" length="0.02"/>
-      </geometry>
-      <material name="green_idler">
-        <color rgba="0.2 1.0 0.2 1.0"/>
-      </material>
+      <geometry><cylinder radius="0.03" length="0.02"/></geometry>
+      <material name="green_idler"><color rgba="0.2 1.0 0.2 1.0"/></material>
+      <origin rpy="1.5708 0 0"/>
     </visual>
   </link>
@@ -120,15 +118,12 @@
     <parent link="base_link"/>
     <child link="left_idler"/>
-    <origin xyz="0.11 0.13 0" rpy="1.5708 0 0"/>
+    <origin xyz="0.11 0.13 0"/>
   </joint>
-  <!-- Right idler wheel -->
+  <!-- Right idler (fixed) -->
   <link name="right_idler">
     <visual>
-      <geometry>
-        <cylinder radius="0.03" length="0.02"/>
-      </geometry>
-      <material name="green_idler">
-        <color rgba="0.2 1.0 0.2 1.0"/>
-      </material>
+      <geometry><cylinder radius="0.03" length="0.02"/></geometry>
+      <material name="green_idler"><color rgba="0.2 1.0 0.2 1.0"/></material>
+      <origin rpy="1.5708 0 0"/>
     </visual>
   </link>
@@ -136,5 +131,5 @@
     <parent link="base_link"/>
     <child link="right_idler"/>
-    <origin xyz="0.11 -0.13 0" rpy="1.5708 0 0"/>
+    <origin xyz="0.11 -0.13 0"/>
   </joint>
 </robot>
