Commit message: Align robot forward axis with physical front

File: src/tank_description/urdf/robot.urdf (robot description, URDF)
Before this commit: robot xiaor_geek_tank_colored, 7 links, 6 joints
Joints:
- joint left_idler_joint: origin xyz=0.11 0.13 0 -> xyz=-0.11 0.13 0
- joint left_wheel_joint: origin xyz=-0.11 0.13 0 -> xyz=0.11 0.13 0
- joint right_idler_joint: origin xyz=0.11 -0.13 0 -> xyz=-0.11 -0.13 0
- joint right_wheel_joint: origin xyz=-0.11 -0.13 0 -> xyz=0.11 -0.13 0

File: src/tank_description/urdf/robot.urdf.xacro (robot description, xacro)
@@ -17,5 +17,5 @@
         <box size="0.16 0.14 0.05"/>
       </geometry>
-      <origin xyz="0.07 0 0.10"/>
+      <origin xyz="-0.07 0 0.10"/>
       <material name="BlueTop">
         <color rgba="0.2 0.2 0.8 1"/>
@@ -27,5 +27,5 @@
         <box size="0.16 0.14 0.05"/>
       </geometry>
-      <origin xyz="0.07 0 0.15"/>
+      <origin xyz="-0.07 0 0.15"/>
       <material name="silver">
         <color rgba="0.7 0.7 0.7 1.0"/>
@@ -90,5 +90,5 @@
     <parent link="base_link"/>
     <child link="left_wheel"/>
-    <origin xyz="-0.11 0.13 0"/>
+    <origin xyz="0.11 0.13 0"/>
     <axis xyz="0 1 0"/>
   </joint>
@@ -104,5 +104,5 @@
     <parent link="base_link"/>
     <child link="right_wheel"/>
-    <origin xyz="-0.11 -0.13 0"/>
+    <origin xyz="0.11 -0.13 0"/>
     <axis xyz="0 1 0"/>
   </joint>
@@ -118,5 +118,5 @@
     <parent link="base_link"/>
     <child link="left_idler"/>
-    <origin xyz="0.11 0.13 0"/>
+    <origin xyz="-0.11 0.13 0"/>
   </joint>
   <!-- Right idler (fixed) -->
@@ -131,5 +131,5 @@
     <parent link="base_link"/>
     <child link="right_idler"/>
-    <origin xyz="0.11 -0.13 0"/>
+    <origin xyz="-0.11 -0.13 0"/>
   </joint>
 </robot>
